Commit message: added gripper camera link to the panda hand

File: robots/panda_hand.urdf (robot description, URDF)
Before this commit: robot panda, 22 links, 21 joints
Links:
- added link gripper_cam, mass 0.2; visual box size=.08 .025 0.01
Joints:
- added joint camera_joint: type fixed, parent panda_hand, child gripper_cam, origin xyz=-0.1 0 0 rpy=1.3  0 -1.57
