Commit message: made the hatch_door red

File: objects/hatch_door.urdf (robot description, URDF)
Before this commit: robot hatch_door, 2 links, 1 joints
Links:
- link door_link: geometry collision box size=0.018 0.29 0.02; collision box size=0.018 0.29 0.02
- link handle_link: geometry collision box size=0.05 0.02 0.02; collision box size=0.05 0.02 0.02
